Commit message: ros_control_namespace -> robot_ns

File: urdf/leo.gazebo.xacro (robot description, xacro)
@@ -4,5 +4,5 @@
   <gazebo>
     <plugin name="gazebo_ros_control" filename="libgazebo_ros_control.so">
-      <robotNamespace>$(arg ros_control_namespace)</robotNamespace>
+      <robotNamespace>$(arg robot_ns)</robotNamespace>
       <robotSimType>gazebo_ros_control/DefaultRobotHWSim</robotSimType>
     </plugin>

File: urdf/leo.urdf.xacro (robot description, xacro)
@@ -2,5 +2,5 @@
 <robot xmlns:xacro="http://www.ros.org/wiki/xacro"
        name="leo">
-  <xacro:arg name="ros_control_namespace" default="leo"/>
+  <xacro:arg name="robot_ns" default="leo"/>
   <xacro:arg name="fixed" default="false"/>
   <xacro:arg name="default_antenna" default="true"/>
@@ -21,5 +21,8 @@
         <mass value="1.387336"/>
         <origin xyz="0 0.01346 -0.06506"/>
-        <inertia ixx="0.002956" ixy="-0.000001489324" ixz="-0.000008103407" iyy="0.02924" iyz="0.00007112" izz="0.02832"/>
+        <inertia
+          ixx="0.002956" ixy="-0.000001489324" ixz="-0.000008103407"
+          iyy="0.02924"  iyz="0.00007112"
+          izz="0.02832"/>
       </inertial>
       <visual>
@@ -40,5 +43,8 @@
         <mass value="0.283642"/>
         <origin xyz="0 0.030026 0"/>
-        <inertia ixx="0.000391" ixy="0.00000123962" ixz="5.52582e-7" iyy="0.0004716" iyz="-0.000002082042" izz="0.000391"/>
+        <inertia
+          ixx="0.000391"  ixy="0.00000123962" ixz="5.52582e-7"
+          iyy="0.0004716" iyz="-0.000002082042"
+          izz="0.000391"/>
       </inertial>
       <visual>
@@ -65,5 +71,8 @@
       <mass value="1.584994"/>
       <origin xyz="-0.019662 0.011643 -0.031802"/>
-      <inertia ixx="0.01042" ixy="0.001177" ixz="-0.0008871" iyy="0.01045" iyz="0.0002226" izz="0.01817"/>
+      <inertia
+        ixx="0.01042" ixy="0.001177" ixz="-0.0008871"
+        iyy="0.01045" iyz="0.0002226"
+        izz="0.01817"/>
     </inertial>
     <visual>
@@ -90,5 +99,8 @@
         <mass value="0.001237"/>
         <origin xyz="0 0 0.028828"/>
-        <inertia ixx="2.5529e-7" ixy="0.0" ixz="0.0" iyy="2.5529e-7" iyz="0.0" izz="1.354e-8"/>
+        <inertia
+          ixx="2.5529e-7" ixy="0.0" ixz="0.0"
+          iyy="2.5529e-7" iyz="0.0"
+          izz="1.354e-8"/>
       </inertial>
       <visual>

Commit message: Rocker differential working

File: urdf/leo.gazebo.xacro (robot description, xacro)
@@ -53,3 +53,12 @@
     </sensor>
   </gazebo>
+  <xacro:unless value="$(arg rockers_fixed)">
+    <gazebo>
+      <plugin name="rocker_differential" filename="libgazebo_differential_plugin.so">
+        <jointA>rocker_L_joint</jointA>
+        <jointB>rocker_R_joint</jointB>
+        <forceConstant>100.0</forceConstant>
+      </plugin>
+    </gazebo>
+  </xacro:unless>
 </robot>

File: urdf/leo.urdf.xacro (robot description, xacro)
@@ -12,5 +12,5 @@
       <parent link="world"/>
       <child link="base_link"/>
-      <origin xyz="0.0 0.0 2.0"/>
+      <origin xyz="0.0 0.0 0"/>
     </joint>
   </xacro:if>
@@ -131,6 +131,6 @@
     <child link="rocker_L_link"/>
     <axis xyz="0 1 0"/>
-    <limit effort="10" lower="-0.24" upper="0.24" velocity="0.5"/> <!-- TODO effort velocity -->
-    <dynamics friction="0.1" damping="0.1"/> <!-- TODO -->
+    <limit effort="100.0" lower="-0.24" upper="0.24" velocity="100.0"/>
+    <dynamics friction="1.0" damping="0.1"/>
   </joint>
   <joint name="rocker_R_joint" type="${rockers_joint_type}">
@@ -139,6 +139,6 @@
     <child link="rocker_R_link"/>
     <axis xyz="0 1 0"/>
-    <limit effort="10" lower="-0.24" upper="0.24" velocity="0.5"/> <!-- TODO effort velocity -->
-    <dynamics friction="0.1" damping="0.1"/> <!-- TODO -->
+    <limit effort="100.0" lower="-0.24" upper="0.24" velocity="100.0"/>
+    <dynamics friction="1.0" damping="0.1"/>
     <mimic joint="rocker_L_joint"/>
   </joint>
@@ -238,3 +238,19 @@
     </actuator>
   </transmission>
+  <xacro:unless value="$(arg rockers_fixed)">
+    <transmission name="rocker_L_trans">
+      <type>transmission_interface/SimpleTransmission</type>
+      <joint name="rocker_L_joint">
+        <hardwareInterface>hardware_interface/EffortJointInterface</hardwareInterface>
+      </joint>
+      <actuator name="rocker_L_virtual_motor"/>
+    </transmission>
+    <transmission name="rocker_R_trans">
+      <type>transmission_interface/SimpleTransmission</type>
+      <joint name="rocker_R_joint">
+        <hardwareInterface>hardware_interface/EffortJointInterface</hardwareInterface>
+      </joint>
+      <actuator name="rocker_R_virtual_motor"/>
+    </transmission>
+  </xacro:unless>
 </robot>
