Commit message: add camera_link to urdf

File: urdf/leo.urdf.xacro (robot description, xacro)
@@ -66,3 +66,9 @@
     <axis xyz="0 0 -1"/>
   </joint>
+  <link name="camera_link"/>
+  <joint name="camera_joint" type="fixed">
+      <origin xyz="0.08 0 -0.04" rpy="${-pi/2 - 0.2} 0 ${-pi/2}"/>
+      <parent link="base_link"/>
+      <child link="camera_link"/>
+  </joint>
 </robot>

Commit message: new model initial

File: urdf/leo.urdf.xacro (robot description, xacro)
@@ -6,16 +6,7 @@
       <origin xyz="0 0 0" rpy="0 0 0" />
       <geometry>
-        <mesh filename="package://leo_description/meshes/base_link.STL"/>
+        <mesh filename="package://leo_description/models/base.dae"/>
       </geometry>
-      <material name="base">
-        <color rgba="0.752941176470588 0.752941176470588 0.752941176470588 1"/>
-      </material>
     </visual>
-    <collision>
-      <origin xyz="0 0 0" rpy="0 0 0"/>
-      <geometry>
-        <mesh filename="package://leo_description/meshes/base_link.STL" />
-      </geometry>
-    </collision>
   </link>
   <xacro:macro name="wheel_link" params="name model">
@@ -24,16 +15,7 @@
         <origin xyz="0 0 0" rpy="0 0 0"/>
         <geometry>
-          <mesh filename="package://leo_description/meshes/wheel_${model}.STL"/>
+          <mesh filename="package://leo_description/models/wheel_${model}.dae"/>
         </geometry>
-        <material name="wheel">
-          <color rgba="0.752941176470588 0.752941176470588 0.752941176470588 1"/>
-        </material>
       </visual>
-      <collision>
-        <origin xyz="0 0 0" rpy="0 0 0"/>
-        <geometry>
-          <mesh filename="package://leo_description/meshes/wheel_${model}.STL"/>
-        </geometry>
-      </collision>
     </link>
   </xacro:macro>
@@ -43,32 +25,32 @@
   <xacro:wheel_link name="RR" model="right"/>
   <joint name="wheel_FL_joint" type="continuous">
-    <origin xyz="0.14211 0.16833 -0.13136" rpy="${pi/2} 0 0"/>
+    <origin xyz="0.1472 0.1114 -0.1353" rpy="0 0 ${pi}"/>
     <parent link="base_link"/>
     <child link="wheel_FL_link"/>
-    <axis xyz="0 0 -1"/>
+    <axis xyz="0 -1 0"/>
   </joint>
   <joint name="wheel_FR_joint" type="continuous">
-    <origin xyz="0.14211 -0.16026 -0.13136" rpy="${pi/2} 0 0"/>
+    <origin xyz="0.1472 -0.1114 -0.1353" rpy="0 0 0"/>
     <parent link="base_link"/>
     <child link="wheel_FR_link"/>
-    <axis xyz="0 0 -1"/>
+    <axis xyz="0 1 0"/>
   </joint>
   <joint name="wheel_RL_joint" type="continuous">
-    <origin xyz="-0.14704 0.16833 -0.13136" rpy="${pi/2} 0 0"/>
+    <origin xyz="-0.1419 0.1114 -0.1353" rpy="0 0 ${pi}"/>
     <parent link="base_link"/>
     <child link="wheel_RL_link"/>
-    <axis xyz="0 0 -1"/>
+    <axis xyz="0 -1 0"/>
   </joint>
   <joint name="wheel_RR_joint" type="continuous">
-    <origin xyz="-0.14704 -0.16026 -0.13136" rpy="${pi/2} 0 0"/>
+    <origin xyz="-0.1419 -0.1114 -0.1353" rpy="0 0 0"/>
     <parent link="base_link"/>
     <child link="wheel_RR_link"/>
-    <axis xyz="0 0 -1"/>
+    <axis xyz="0 1 0"/>
   </joint>
-  <link name="camera_link"/>
+  <link name="camera_frame"/>
   <joint name="camera_joint" type="fixed">
-      <origin xyz="0.08 0 -0.04" rpy="${-pi/2 - 0.2} 0 ${-pi/2}"/>
+      <origin xyz="0.0971 0 -0.0427" rpy="${-pi/2 - 0.2094} 0 ${-pi/2}"/>
       <parent link="base_link"/>
-      <child link="camera_link"/>
+      <child link="camera_frame"/>
   </joint>
 </robot>

Commit message: Completely replace meshes with more optimized ones, add joints for rockers and antenna, add mass and intertial properties

File: urdf/leo.urdf.xacro (robot description, xacro)
@@ -1,13 +1,27 @@
 <?xml version="1.0" encoding="utf-8"?>
 <robot xmlns:xacro="http://www.ros.org/wiki/xacro"
-       name="leo_description">
-  <link name="base_link">
-    <visual>
-      <origin xyz="0 0 0" rpy="0 0 0" />
-      <geometry>
-        <mesh filename="package://leo_description/models/base.dae"/>
-      </geometry>
-    </visual>
-  </link>
+       name="leo">
+  <!-- MACROS -->
+  <xacro:macro name="rocker_link" params="name">
+    <link name="rocker_${name}_link">
+    <inertial>
+      <mass value="1.387336"/>
+      <origin xyz="0 0.01346 -0.06506"/>
+      <inertia ixx="0.002956" ixy="-0.000001489324" ixz="-0.000008103407" iyy="0.02924" iyz="0.00007112" izz="0.02832"/>
+    </inertial>
+      <visual>
+        <origin xyz="0 0 0" rpy="0 0 0"/>
+        <geometry>
+          <mesh filename="package://leo_description/models/Rocker.dae"/>
+        </geometry>
+      </visual>
+      <collision>
+        <origin xyz="0 0 0" rpy="0 0 0"/>
+        <geometry>
+          <mesh filename="package://leo_description/models/Rocker.dae"/>
+        </geometry>
+      </collision>
+    </link>
+  </xacro:macro>
   <xacro:macro name="wheel_link" params="name model">
     <link name="wheel_${name}_link">
@@ -15,38 +29,103 @@
         <origin xyz="0 0 0" rpy="0 0 0"/>
         <geometry>
-          <mesh filename="package://leo_description/models/wheel_${model}.dae"/>
+          <mesh filename="package://leo_description/models/Wheel${model}.dae"/>
         </geometry>
       </visual>
     </link>
   </xacro:macro>
-  <xacro:wheel_link name="FL" model="left"/>
-  <xacro:wheel_link name="FR" model="right"/>
-  <xacro:wheel_link name="RL" model="left"/>
-  <xacro:wheel_link name="RR" model="right"/>
+  <!-- LINKS -->
+  <link name="base_link">
+    <inertial>
+      <mass value="1.584994"/>
+      <origin xyz="-0.019662 0.011643 -0.031802"/>
+      <inertia ixx="0.01042" ixy="0.001177" ixz="-0.0008871" iyy="0.01045" iyz="0.0002226" izz="0.01817"/>
+    </inertial>
+    <visual>
+      <origin xyz="0 0 0" rpy="0 0 0" />
+      <geometry>
+        <mesh filename="package://leo_description/models/Chassis.dae"/>
+      </geometry>
+    </visual>
+    <collision>
+      <origin xyz="0 0 0" rpy="0 0 0" />
+      <geometry>
+        <mesh filename="package://leo_description/models/Chassis.dae"/>
+      </geometry>
+    </collision>
+  </link>
+  <xacro:rocker_link name="L"/>
+  <xacro:rocker_link name="R"/>
+  <xacro:wheel_link name="FL" model="A"/>
+  <xacro:wheel_link name="RL" model="A"/>
+  <xacro:wheel_link name="FR" model="B"/>
+  <xacro:wheel_link name="RR" model="B"/>
+  <link name="antenna_link">
+    <inertial>
+      <mass value="0.001237"/>
+      <origin xyz="0 0 0.028828"/>
+      <inertia ixx="2.5529e-7" ixy="0.0" ixz="0.0" iyy="2.5529e-7" iyz="0.0" izz="1.354e-8"/>
+    </inertial>
+    <visual>
+      <origin xyz="0 0 0"/>
+      <geometry>
+        <mesh filename="package://leo_description/models/Antenna.dae"/>
+      </geometry>
+    </visual>
+    <collision>
+      <origin xyz="0 0 0.028"/>
+      <geometry>
+        <cylinder radius="0.0055" length="0.056"/>
+      </geometry>
+    </collision>
+  </link>
+  <link name="camera_frame"/>
+  <!-- JOINTS -->
+  <joint name="rocker_L_joint" type="revolute">
+    <origin xyz="0.00263 0.14167 -0.04731" rpy="0 0 ${pi}"/>
+    <parent link="base_link"/>
+    <child link="rocker_L_link"/>
+    <axis xyz="0 1 0"/>
+    <limit effort="10" lower="-0.3" upper="0.3" velocity="0.5"/> <!-- TODO -->
+  </joint>
+  <joint name="rocker_R_joint" type="revolute">
+    <origin xyz="0.00263 -0.14167 -0.04731" rpy="0 0 0"/>
+    <parent link="base_link"/>
+    <child link="rocker_R_link"/>
+    <axis xyz="0 1 0"/>
+    <limit effort="10" lower="-0.3" upper="0.3" velocity="0.5"/> <!-- TODO -->
+  </joint>
   <joint name="wheel_FL_joint" type="continuous">
-    <origin xyz="0.1472 0.1114 -0.1353" rpy="0 0 ${pi}"/>
-    <parent link="base_link"/>
+    <origin xyz="-0.15256 -0.08214 -0.08802" rpy="0 0 0"/>
+    <parent link="rocker_L_link"/>
     <child link="wheel_FL_link"/>
     <axis xyz="0 -1 0"/>
+    <limit effort="10" velocity="1.0"/> <!-- TODO -->
+  </joint>
+  <joint name="wheel_RL_joint" type="continuous">
+    <origin xyz="0.15256 -0.08214 -0.08802" rpy="0 0 0"/>
+    <parent link="rocker_L_link"/>
+    <child link="wheel_RL_link"/>
+    <axis xyz="0 -1 0"/>
+    <limit effort="10" velocity="1.0"/> <!-- TODO -->
   </joint>
   <joint name="wheel_FR_joint" type="continuous">
-    <origin xyz="0.1472 -0.1114 -0.1353" rpy="0 0 0"/>
-    <parent link="base_link"/>
+    <origin xyz="0.15256 -0.08214 -0.08802" rpy="0 0 0"/>
+    <parent link="rocker_R_link"/>
     <child link="wheel_FR_link"/>
     <axis xyz="0 1 0"/>
-  </joint>
-  <joint name="wheel_RL_joint" type="continuous">
-    <origin xyz="-0.1419 0.1114 -0.1353" rpy="0 0 ${pi}"/>
-    <parent link="base_link"/>
-    <child link="wheel_RL_link"/>
-    <axis xyz="0 -1 0"/>
+    <limit effort="10" velocity="1.0"/> <!-- TODO -->
   </joint>
   <joint name="wheel_RR_joint" type="continuous">
-    <origin xyz="-0.1419 -0.1114 -0.1353" rpy="0 0 0"/>
-    <parent link="base_link"/>
+    <origin xyz="-0.15256 -0.08214 -0.08802" rpy="0 0 0"/>
+    <parent link="rocker_R_link"/>
     <child link="wheel_RR_link"/>
     <axis xyz="0 1 0"/>
+    <limit effort="10" velocity="1.0"/> <!-- TODO -->
   </joint>
-  <link name="camera_frame"/>
+  <joint name="antenna_joint" type="fixed">
+      <origin xyz="-0.0052 0.056 -0.0065" rpy="0 0 0"/>
+      <parent link="base_link"/>
+      <child link="antenna_link"/>
+  </joint>
   <joint name="camera_joint" type="fixed">
       <origin xyz="0.0971 0 -0.0427" rpy="${-pi/2 - 0.2094} 0 ${-pi/2}"/>

Commit message: Add inertial properties to wheels, change rocker joint limits and make the right rocker joint mimic the left one

File: urdf/leo.urdf.xacro (robot description, xacro)
@@ -11,5 +11,4 @@
     </inertial>
       <visual>
-        <origin xyz="0 0 0" rpy="0 0 0"/>
         <geometry>
           <mesh filename="package://leo_description/models/Rocker.dae"/>
@@ -17,5 +16,4 @@
       </visual>
       <collision>
-        <origin xyz="0 0 0" rpy="0 0 0"/>
         <geometry>
           <mesh filename="package://leo_description/models/Rocker.dae"/>
@@ -26,10 +24,20 @@
   <xacro:macro name="wheel_link" params="name model">
     <link name="wheel_${name}_link">
+      <inertial>
+        <mass value="0.283642"/>
+        <origin xyz="0 0.030026 0"/>
+        <inertia ixx="0.000391" ixy="0.00000123962" ixz="5.52582e-7" iyy="0.0004716" iyz="-0.000002082042" izz="0.000391"/>
+      </inertial>
       <visual>
-        <origin xyz="0 0 0" rpy="0 0 0"/>
         <geometry>
           <mesh filename="package://leo_description/models/Wheel${model}.dae"/>
         </geometry>
       </visual>
+      <collision>
+        <origin xyz="0 0.04485 0" rpy="${pi/2} 0 0"/>
+        <geometry>
+          <cylinder radius="0.06" length="0.07"/>
+        </geometry>
+      </collision>
     </link>
   </xacro:macro>
@@ -42,5 +50,4 @@
     </inertial>
     <visual>
-      <origin xyz="0 0 0" rpy="0 0 0" />
       <geometry>
         <mesh filename="package://leo_description/models/Chassis.dae"/>
@@ -48,5 +55,4 @@
     </visual>
     <collision>
-      <origin xyz="0 0 0" rpy="0 0 0" />
       <geometry>
         <mesh filename="package://leo_description/models/Chassis.dae"/>
@@ -67,5 +73,4 @@
     </inertial>
     <visual>
-      <origin xyz="0 0 0"/>
       <geometry>
         <mesh filename="package://leo_description/models/Antenna.dae"/>
@@ -86,5 +91,5 @@
     <child link="rocker_L_link"/>
     <axis xyz="0 1 0"/>
-    <limit effort="10" lower="-0.3" upper="0.3" velocity="0.5"/> <!-- TODO -->
+    <limit effort="10" lower="-0.24" upper="0.24" velocity="0.5"/> <!-- TODO -->
   </joint>
   <joint name="rocker_R_joint" type="revolute">
@@ -93,5 +98,6 @@
     <child link="rocker_R_link"/>
     <axis xyz="0 1 0"/>
-    <limit effort="10" lower="-0.3" upper="0.3" velocity="0.5"/> <!-- TODO -->
+    <limit effort="10" lower="-0.24" upper="0.24" velocity="0.5"/> <!-- TODO -->
+    <mimic joint="rocker_L_joint"/>
   </joint>
   <joint name="wheel_FL_joint" type="continuous">

Commit message: Change max wheel velocity

File: urdf/leo.urdf.xacro (robot description, xacro)
@@ -106,5 +106,5 @@
     <child link="wheel_FL_link"/>
     <axis xyz="0 -1 0"/>
-    <limit effort="10" velocity="1.0"/> <!-- TODO -->
+    <limit effort="10" velocity="6.0"/> <!-- TODO -->
   </joint>
   <joint name="wheel_RL_joint" type="continuous">
@@ -113,5 +113,5 @@
     <child link="wheel_RL_link"/>
     <axis xyz="0 -1 0"/>
-    <limit effort="10" velocity="1.0"/> <!-- TODO -->
+    <limit effort="10" velocity="6.0"/> <!-- TODO -->
   </joint>
   <joint name="wheel_FR_joint" type="continuous">
@@ -120,5 +120,5 @@
     <child link="wheel_FR_link"/>
     <axis xyz="0 1 0"/>
-    <limit effort="10" velocity="1.0"/> <!-- TODO -->
+    <limit effort="10" velocity="6.0"/> <!-- TODO -->
   </joint>
   <joint name="wheel_RR_joint" type="continuous">
@@ -127,5 +127,5 @@
     <child link="wheel_RR_link"/>
     <axis xyz="0 1 0"/>
-    <limit effort="10" velocity="1.0"/> <!-- TODO -->
+    <limit effort="10" velocity="6.0"/> <!-- TODO -->
   </joint>
   <joint name="antenna_joint" type="fixed">

Commit message: Make the antenna link optional by adding  argument to the xacro file

File: urdf/leo.urdf.xacro (robot description, xacro)
@@ -2,4 +2,5 @@
 <robot xmlns:xacro="http://www.ros.org/wiki/xacro"
        name="leo">
+  <xacro:arg name="default_antenna" default="true"/>
   <!-- MACROS -->
   <xacro:macro name="rocker_link" params="name">
@@ -66,22 +67,24 @@
   <xacro:wheel_link name="FR" model="B"/>
   <xacro:wheel_link name="RR" model="B"/>
-  <link name="antenna_link">
-    <inertial>
-      <mass value="0.001237"/>
-      <origin xyz="0 0 0.028828"/>
-      <inertia ixx="2.5529e-7" ixy="0.0" ixz="0.0" iyy="2.5529e-7" iyz="0.0" izz="1.354e-8"/>
-    </inertial>
-    <visual>
-      <geometry>
-        <mesh filename="package://leo_description/models/Antenna.dae"/>
-      </geometry>
-    </visual>
-    <collision>
-      <origin xyz="0 0 0.028"/>
-      <geometry>
-        <cylinder radius="0.0055" length="0.056"/>
-      </geometry>
-    </collision>
-  </link>
+  <xacro:if value="$(arg default_antenna)">
+    <link name="antenna_link">
+      <inertial>
+        <mass value="0.001237"/>
+        <origin xyz="0 0 0.028828"/>
+        <inertia ixx="2.5529e-7" ixy="0.0" ixz="0.0" iyy="2.5529e-7" iyz="0.0" izz="1.354e-8"/>
+      </inertial>
+      <visual>
+        <geometry>
+          <mesh filename="package://leo_description/models/Antenna.dae"/>
+        </geometry>
+      </visual>
+      <collision>
+        <origin xyz="0 0 0.028"/>
+        <geometry>
+          <cylinder radius="0.0055" length="0.056"/>
+        </geometry>
+      </collision>
+    </link>
+  </xacro:if>
   <link name="camera_frame"/>
   <!-- JOINTS -->
@@ -129,9 +132,11 @@
     <limit effort="10" velocity="6.0"/> <!-- TODO -->
   </joint>
-  <joint name="antenna_joint" type="fixed">
-      <origin xyz="-0.0052 0.056 -0.0065" rpy="0 0 0"/>
-      <parent link="base_link"/>
-      <child link="antenna_link"/>
-  </joint>
+  <xacro:if value="$(arg default_antenna)">
+    <joint name="antenna_joint" type="fixed">
+        <origin xyz="-0.0052 0.056 -0.0065" rpy="0 0 0"/>
+        <parent link="base_link"/>
+        <child link="antenna_link"/>
+    </joint>
+  </xacro:if>
   <joint name="camera_joint" type="fixed">
       <origin xyz="0.0971 0 -0.0427" rpy="${-pi/2 - 0.2094} 0 ${-pi/2}"/>

Commit message: Add  argument which lets the user choose whether to use fixed or revolute joints for rocker links

File: urdf/leo.urdf.xacro (robot description, xacro)
@@ -3,4 +3,5 @@
        name="leo">
   <xacro:arg name="default_antenna" default="true"/>
+  <xacro:arg name="rockers_fixed" default="true"/>
   <!-- MACROS -->
   <xacro:macro name="rocker_link" params="name">
@@ -16,5 +17,5 @@
         </geometry>
       </visual>
-      <collision>
+      <collision> <!-- TODO -->
         <geometry>
           <mesh filename="package://leo_description/models/Rocker.dae"/>
@@ -35,5 +36,5 @@
         </geometry>
       </visual>
-      <collision>
+      <collision> <!-- TODO -->
         <origin xyz="0 0.04485 0" rpy="${pi/2} 0 0"/>
         <geometry>
@@ -55,5 +56,5 @@
       </geometry>
     </visual>
-    <collision>
+    <collision> <!-- TODO -->
       <geometry>
         <mesh filename="package://leo_description/models/Chassis.dae"/>
@@ -61,4 +62,5 @@
     </collision>
   </link>
+  <link name="base_footprint"/>
   <xacro:rocker_link name="L"/>
   <xacro:rocker_link name="R"/>
@@ -89,17 +91,25 @@
   <link name="camera_frame"/>
   <!-- JOINTS -->
-  <joint name="rocker_L_joint" type="revolute">
+  <xacro:if value="$(arg rockers_fixed)">
+    <xacro:property name="rockers_joint_type" value="fixed"/>
+  </xacro:if>
+  <xacro:unless value="$(arg rockers_fixed)">
+    <xacro:property name="rockers_joint_type" value="revolute"/>
+  </xacro:unless>
+  <joint name="rocker_L_joint" type="${rockers_joint_type}">
     <origin xyz="0.00263 0.14167 -0.04731" rpy="0 0 ${pi}"/>
     <parent link="base_link"/>
     <child link="rocker_L_link"/>
     <axis xyz="0 1 0"/>
-    <limit effort="10" lower="-0.24" upper="0.24" velocity="0.5"/> <!-- TODO -->
+    <limit effort="10" lower="-0.24" upper="0.24" velocity="0.5"/> <!-- TODO effort velocity -->
+    <dynamics friction="0.1" damping="0.1"/> <!-- TODO -->
   </joint>
-  <joint name="rocker_R_joint" type="revolute">
+  <joint name="rocker_R_joint" type="${rockers_joint_type}">
     <origin xyz="0.00263 -0.14167 -0.04731" rpy="0 0 0"/>
     <parent link="base_link"/>
     <child link="rocker_R_link"/>
     <axis xyz="0 1 0"/>
-    <limit effort="10" lower="-0.24" upper="0.24" velocity="0.5"/> <!-- TODO -->
+    <limit effort="10" lower="-0.24" upper="0.24" velocity="0.5"/> <!-- TODO effort velocity -->
+    <dynamics friction="0.1" damping="0.1"/> <!-- TODO -->
     <mimic joint="rocker_L_joint"/>
   </joint>
@@ -109,5 +119,6 @@
     <child link="wheel_FL_link"/>
     <axis xyz="0 -1 0"/>
-    <limit effort="10" velocity="6.0"/> <!-- TODO -->
+    <limit effort="10" velocity="6.0"/> <!-- TODO effort -->
+    <dynamics friction="0.1" damping="0.1"/> <!-- TODO -->
   </joint>
   <joint name="wheel_RL_joint" type="continuous">
@@ -116,19 +127,22 @@
     <child link="wheel_RL_link"/>
     <axis xyz="0 -1 0"/>
-    <limit effort="10" velocity="6.0"/> <!-- TODO -->
+    <limit effort="10" velocity="6.0"/> <!-- TODO effort -->
+    <dynamics friction="0.1" damping="0.1"/> <!-- TODO -->
   </joint>
   <joint name="wheel_FR_joint" type="continuous">
-    <origin xyz="0.15256 -0.08214 -0.08802" rpy="0 0 0"/>
+    <origin xyz="-0.15256 -0.08214 -0.08802" rpy="0 0 0"/>
     <parent link="rocker_R_link"/>
     <child link="wheel_FR_link"/>
     <axis xyz="0 1 0"/>
-    <limit effort="10" velocity="6.0"/> <!-- TODO -->
+    <limit effort="10" velocity="6.0"/> <!-- TODO effort -->
+    <dynamics friction="0.1" damping="0.1"/> <!-- TODO -->
   </joint>
   <joint name="wheel_RR_joint" type="continuous">
-    <origin xyz="-0.15256 -0.08214 -0.08802" rpy="0 0 0"/>
+    <origin xyz="0.15256 -0.08214 -0.08802" rpy="0 0 0"/>
     <parent link="rocker_R_link"/>
     <child link="wheel_RR_link"/>
     <axis xyz="0 1 0"/>
-    <limit effort="10" velocity="6.0"/> <!-- TODO -->
+    <limit effort="10" velocity="6.0"/> <!-- TODO effort -->
+    <dynamics friction="0.1" damping="0.1"/> <!-- TODO -->
   </joint>
   <xacro:if value="$(arg default_antenna)">
@@ -144,3 +158,8 @@
       <child link="camera_frame"/>
   </joint>
+  <joint name="footprint_joint" type="fixed">
+      <origin xyz="0 0 -0.19783" rpy="0 0 0"/>
+      <parent link="base_link"/>
+      <child link="base_footprint"/>
+  </joint>
 </robot>

Commit message: Add low-poly outline models for collision geometry

File: urdf/leo.urdf.xacro (robot description, xacro)
@@ -7,9 +7,9 @@
   <xacro:macro name="rocker_link" params="name">
     <link name="rocker_${name}_link">
-    <inertial>
-      <mass value="1.387336"/>
-      <origin xyz="0 0.01346 -0.06506"/>
-      <inertia ixx="0.002956" ixy="-0.000001489324" ixz="-0.000008103407" iyy="0.02924" iyz="0.00007112" izz="0.02832"/>
-    </inertial>
+      <inertial>
+        <mass value="1.387336"/>
+        <origin xyz="0 0.01346 -0.06506"/>
+        <inertia ixx="0.002956" ixy="-0.000001489324" ixz="-0.000008103407" iyy="0.02924" iyz="0.00007112" izz="0.02832"/>
+      </inertial>
       <visual>
         <geometry>
@@ -17,7 +17,7 @@
         </geometry>
       </visual>
-      <collision> <!-- TODO -->
+      <collision>
         <geometry>
-          <mesh filename="package://leo_description/models/Rocker.dae"/>
+          <mesh filename="package://leo_description/models/Rocker_outline.stl"/>
         </geometry>
       </collision>
@@ -36,8 +36,13 @@
         </geometry>
       </visual>
-      <collision> <!-- TODO -->
+      <collision>
         <origin xyz="0 0.04485 0" rpy="${pi/2} 0 0"/>
         <geometry>
-          <cylinder radius="0.06" length="0.07"/>
+          <cylinder radius="0.0625" length="0.07"/>
+        </geometry>
+      </collision>
+      <collision>
+        <geometry>
+          <mesh filename="package://leo_description/models/Wheel_outline.stl"/>
         </geometry>
       </collision>
@@ -56,7 +61,7 @@
       </geometry>
     </visual>
-    <collision> <!-- TODO -->
+    <collision>
       <geometry>
-        <mesh filename="package://leo_description/models/Chassis.dae"/>
+        <mesh filename="package://leo_description/models/Chassis_outline.stl"/>
       </geometry>
     </collision>
