Commit message: Add transmission tags and gazebo_ros_control plugin

File: urdf/leo.urdf.xacro (robot description, xacro)
@@ -2,6 +2,17 @@
 <robot xmlns:xacro="http://www.ros.org/wiki/xacro"
        name="leo">
+  <xacro:arg name="ros_control_namespace" default="leo"/>
+  <xacro:arg name="fixed" default="false"/>
   <xacro:arg name="default_antenna" default="true"/>
   <xacro:arg name="rockers_fixed" default="true"/>
+  <xacro:include filename="$(find leo_description)/urdf/leo.gazebo.xacro"/>
+  <xacro:if value="$(arg fixed)">
+    <link name="world"/>
+    <joint name="fixed" type="fixed">
+      <parent link="world"/>
+      <child link="base_link"/>
+      <origin xyz="0.0 0.0 2.0"/>
+    </joint>
+  </xacro:if>
   <!-- MACROS -->
   <xacro:macro name="rocker_link" params="name">
@@ -168,3 +179,44 @@
       <child link="base_footprint"/>
   </joint>
+  <!-- TRANSMISSIONS -->
+  <transmission name="wheel_FL_trans">
+    <type>transmission_interface/SimpleTransmission</type>
+    <joint name="wheel_FL_joint">
+      <hardwareInterface>hardware_interface/VelocityJointInterface</hardwareInterface>
+    </joint>
+    <actuator name="wheel_FL_motor">
+      <mechanicalReduction>1</mechanicalReduction>
+      <hardwareInterface>hardware_interface/VelocityJointInterface</hardwareInterface>
+    </actuator>
+  </transmission>
+  <transmission name="wheel_RL_trans">
+    <type>transmission_interface/SimpleTransmission</type>
+    <joint name="wheel_RL_joint">
+      <hardwareInterface>hardware_interface/VelocityJointInterface</hardwareInterface>
+    </joint>
+    <actuator name="wheel_RL_motor">
+      <mechanicalReduction>1</mechanicalReduction>
+      <hardwareInterface>hardware_interface/VelocityJointInterface</hardwareInterface>
+    </actuator>
+  </transmission>
+  <transmission name="wheel_FR_trans">
+    <type>transmission_interface/SimpleTransmission</type>
+    <joint name="wheel_FR_joint">
+      <hardwareInterface>hardware_interface/VelocityJointInterface</hardwareInterface>
+    </joint>
+    <actuator name="wheel_FR_motor">
+      <mechanicalReduction>1</mechanicalReduction>
+      <hardwareInterface>hardware_interface/VelocityJointInterface</hardwareInterface>
+    </actuator>
+  </transmission>
+  <transmission name="wheel_RR_trans">
+    <type>transmission_interface/SimpleTransmission</type>
+    <joint name="wheel_RR_joint">
+      <hardwareInterface>hardware_interface/VelocityJointInterface</hardwareInterface>
+    </joint>
+    <actuator name="wheel_RR_motor">
+      <mechanicalReduction>1</mechanicalReduction>
+      <hardwareInterface>hardware_interface/VelocityJointInterface</hardwareInterface>
+    </actuator>
+  </transmission>
 </robot>

Commit message: Add camera_optical_frame link which uses camera coordinate convention

File: urdf/leo.urdf.xacro (robot description, xacro)
@@ -118,4 +118,5 @@
   </xacro:if>
   <link name="camera_frame"/>
+  <link name="camera_optical_frame"/>
   <!-- JOINTS -->
   <xacro:if value="$(arg rockers_fixed)">
@@ -176,18 +177,23 @@
   <xacro:if value="$(arg default_antenna)">
     <joint name="antenna_joint" type="fixed">
-        <origin xyz="-0.0052 0.056 -0.0065" rpy="0 0 0"/>
-        <parent link="base_link"/>
-        <child link="antenna_link"/>
+      <origin xyz="-0.0052 0.056 -0.0065" rpy="0 0 0"/>
+      <parent link="base_link"/>
+      <child link="antenna_link"/>
     </joint>
   </xacro:if>
   <joint name="camera_joint" type="fixed">
-      <origin xyz="0.0971 0 -0.0427" rpy="${-pi/2 - 0.2094} 0 ${-pi/2}"/>
-      <parent link="base_link"/>
-      <child link="camera_frame"/>
+    <origin xyz="0.0971 0 -0.0427" rpy="0 0.2094 0"/>
+    <parent link="base_link"/>
+    <child link="camera_frame"/>
+  </joint>
+  <joint name="camera_optical_joint" type="fixed">
+    <origin xyz="0 0 0" rpy="-${pi/2} 0.0 -${pi/2}"/>
+    <parent link="camera_frame"/>
+    <child link="camera_optical_frame"/>
   </joint>
   <joint name="footprint_joint" type="fixed">
-      <origin xyz="0 0 -0.19783" rpy="0 0 0"/>
-      <parent link="base_link"/>
-      <child link="base_footprint"/>
+    <origin xyz="0 0 -0.19783" rpy="0 0 0"/>
+    <parent link="base_link"/>
+    <child link="base_footprint"/>
   </joint>
   <!-- TRANSMISSIONS -->

Commit message: Tune the friction and effort limit values for wheel joints

File: urdf/leo.urdf.xacro (robot description, xacro)
@@ -148,6 +148,6 @@
     <child link="wheel_FL_link"/>
     <axis xyz="0 -1 0"/>
-    <limit effort="10" velocity="6.0"/> <!-- TODO effort -->
-    <dynamics friction="0.1" damping="0.1"/> <!-- TODO -->
+    <limit effort="5.0" velocity="6.0"/>
+    <dynamics friction="0.3125" damping="0.1"/>
   </joint>
   <joint name="wheel_RL_joint" type="continuous">
@@ -156,6 +156,6 @@
     <child link="wheel_RL_link"/>
     <axis xyz="0 -1 0"/>
-    <limit effort="10" velocity="6.0"/> <!-- TODO effort -->
-    <dynamics friction="0.1" damping="0.1"/> <!-- TODO -->
+    <limit effort="5.0" velocity="6.0"/>
+    <dynamics friction="0.3125" damping="0.1"/>
   </joint>
   <joint name="wheel_FR_joint" type="continuous">
@@ -164,6 +164,6 @@
     <child link="wheel_FR_link"/>
     <axis xyz="0 1 0"/>
-    <limit effort="10" velocity="6.0"/> <!-- TODO effort -->
-    <dynamics friction="0.1" damping="0.1"/> <!-- TODO -->
+    <limit effort="5.0" velocity="6.0"/>
+    <dynamics friction="0.3125" damping="0.1"/>
   </joint>
   <joint name="wheel_RR_joint" type="continuous">
@@ -172,6 +172,6 @@
     <child link="wheel_RR_link"/>
     <axis xyz="0 1 0"/>
-    <limit effort="10" velocity="6.0"/> <!-- TODO effort -->
-    <dynamics friction="0.1" damping="0.1"/> <!-- TODO -->
+    <limit effort="5.0" velocity="6.0"/>
+    <dynamics friction="0.3125" damping="0.1"/>
   </joint>
   <xacro:if value="$(arg default_antenna)">

Commit message: Reduce the effort limits on wheels

File: urdf/leo.urdf.xacro (robot description, xacro)
@@ -148,5 +148,5 @@
     <child link="wheel_FL_link"/>
     <axis xyz="0 -1 0"/>
-    <limit effort="5.0" velocity="6.0"/>
+    <limit effort="2.0" velocity="6.0"/>
     <dynamics friction="0.3125" damping="0.1"/>
   </joint>
@@ -156,5 +156,5 @@
     <child link="wheel_RL_link"/>
     <axis xyz="0 -1 0"/>
-    <limit effort="5.0" velocity="6.0"/>
+    <limit effort="2.0" velocity="6.0"/>
     <dynamics friction="0.3125" damping="0.1"/>
   </joint>
@@ -164,5 +164,5 @@
     <child link="wheel_FR_link"/>
     <axis xyz="0 1 0"/>
-    <limit effort="5.0" velocity="6.0"/>
+    <limit effort="2.0" velocity="6.0"/>
     <dynamics friction="0.3125" damping="0.1"/>
   </joint>
@@ -172,5 +172,5 @@
     <child link="wheel_RR_link"/>
     <axis xyz="0 1 0"/>
-    <limit effort="5.0" velocity="6.0"/>
+    <limit effort="2.0" velocity="6.0"/>
     <dynamics friction="0.3125" damping="0.1"/>
   </joint>

Commit message: Modify wheel friction parameters and collision models

File: urdf/leo.urdf.xacro (robot description, xacro)
@@ -56,5 +56,11 @@
         <origin xyz="0 0.04485 0" rpy="${pi/2} 0 0"/>
         <geometry>
-          <cylinder radius="0.0625" length="0.07"/>
+          <cylinder radius="0.057" length="0.07"/>
+        </geometry>
+      </collision>
+      <collision>
+        <origin xyz="0 0.04485 0" rpy="${pi/2} 0 0"/>
+        <geometry>
+          <cylinder radius="0.0625" length="0.04"/>
         </geometry>
       </collision>
