Commit message: leo_description: Add fixed option to leo_gazebo macro

File: leo_description/urdf/leo_gazebo.urdf.xacro (robot description, xacro)
@@ -2,6 +2,8 @@
 <robot xmlns:xacro="http://ros.org/wiki/xacro"
        name="leo_gazebo">
+  <xacro:arg name="fixed" default="false"/>
   <xacro:arg name="robot_ns" default=""/>
   <xacro:include filename="$(find leo_description)/urdf/leo_macros.xacro"/>
-  <xacro:leo_gazebo robot_ns="$(arg robot_ns)"/>
+  <xacro:leo_gazebo robot_ns="$(arg robot_ns)"
+                    fixed="$(arg fixed)"/>
 </robot>

File: leo_description/urdf/leo_macros.xacro (robot description, xacro)
@@ -196,7 +196,9 @@
   <!-- LEO GAZEBO -->
   <xacro:macro name="leo_gazebo"
-               params="default_antenna:=true robot_ns:=''">
+               params="default_antenna:=true
+                       fixed:=false
+                       robot_ns:=''">
     <xacro:property name="link_prefix" value=""/>
-    <xacro:if value="${robot_ns != ''}">
+    <xacro:if value="${robot_ns != '' and robot_ns != '/'}">
       <xacro:property name="link_prefix" value="${robot_ns}/"/>
     </xacro:if>
@@ -204,4 +206,12 @@
                rockers_fixed="false"
                link_prefix="${link_prefix}"/>
+    <xacro:if value="${fixed}">
+      <link name="world"/>
+      <joint name="fixed" type="fixed">
+        <parent link="world"/>
+        <child link="${link_prefix}base_footprint"/>
+        <origin xyz="0.0 0.0 0"/>
+      </joint>
+    </xacro:if>
     <!-- rocker ODE properties -->
     <gazebo reference="${link_prefix}rocker_L_link">
@@ -295,5 +305,5 @@
     <!-- rocker differential -->
     <gazebo>
-      <plugin name="rocker_differential" filename="libgazebo_differential_plugin.so">
+      <plugin name="rocker_differential" filename="libleo_gazebo_differential_plugin.so">
         <jointA>rocker_L_joint</jointA>
         <jointB>rocker_R_joint</jointB>
