Commit message: added macros in xacro robot description for mecanum wheels
Signed-off-by: Aleksander Szymański <bitterisland6@gmail.com>

File: leo_description/urdf/macros.xacro (robot description, xacro)
@@ -7,5 +7,6 @@
                        link_prefix:=''
                        joint_prefix:=''
-                       imu_translation:='0.0628 -0.0314 -0.0393'">
+                       imu_translation:='0.0628 -0.0314 -0.0393'
+                       mecanum_wheels:=false">
     <xacro:macro name="rocker_link" params="name">
       <link name="${link_prefix}rocker_${name}_link">
@@ -60,4 +61,32 @@
           <geometry>
             <mesh filename="package://leo_description/models/Wheel_outline.stl"/>
+          </geometry>
+        </collision>
+      </link>
+    </xacro:macro>
+    <xacro:macro name="mecanum_wheel_link" params="name model">
+      <link name="${link_prefix}wheel_${name}_link">
+        <inertial>
+          <mass value="0.672214"/>
+          <origin xyz="0 -0.036852 0"/>
+          <inertia
+            ixx="0.0009778"  ixy="-8.10228e-7" ixz="3.2e-11"
+            iyy="0.001321" iyz="5.7e-11"
+            izz="0.0009773"/>
+        </inertial>
+        <visual>
+          <geometry>
+            <mesh filename="package://leo_description/models/WheelMecanum${model}.dae"/>
+          </geometry>
+        </visual>
+        <collision>
+          <origin xyz="0 -0.0317 0" rpy="${pi/2} 0 0"/>
+          <geometry>
+            <cylinder radius="0.0635" length="0.0515"/>
+          </geometry>
+        </collision>
+        <collision>
+          <geometry>
+            <mesh filename="package://leo_description/models/Mecanum_wheel_outline.stl"/>
           </geometry>
         </collision>
@@ -90,8 +119,16 @@
     <xacro:rocker_link name="L"/>
     <xacro:rocker_link name="R"/>
-    <xacro:wheel_link name="FL" model="A"/>
-    <xacro:wheel_link name="RL" model="A"/>
-    <xacro:wheel_link name="FR" model="B"/>
-    <xacro:wheel_link name="RR" model="B"/>
+    <xacro:if value="${mecanum_wheels}">
+      <xacro:mecanum_wheel_link name="FL" model="B"/>
+      <xacro:mecanum_wheel_link name="RL" model="A"/>
+      <xacro:mecanum_wheel_link name="FR" model="A"/>
+      <xacro:mecanum_wheel_link name="RR" model="B"/>
+    </xacro:if>
+    <xacro:unless value="${mecanum_wheels}">
+      <xacro:wheel_link name="FL" model="A"/>
+      <xacro:wheel_link name="RL" model="A"/>
+      <xacro:wheel_link name="FR" model="B"/>
+      <xacro:wheel_link name="RR" model="B"/>
+    </xacro:unless>
     <xacro:if value="${default_antenna}">
       <link name="${link_prefix}antenna_link">
@@ -152,5 +189,10 @@
     </joint>
     <joint name="${joint_prefix}wheel_FL_joint" type="continuous">
-      <origin xyz="-0.15256 -0.08214 -0.08802" rpy="0 0 0"/>
+      <xacro:if value="${mecanum_wheels}">
+        <origin xyz="-0.15256 -0.00884 -0.08802" rpy="0 0 0"/>
+      </xacro:if>
+      <xacro:unless value="${mecanum_wheels}">
+        <origin xyz="-0.15256 -0.08214 -0.08802" rpy="0 0 0"/>
+      </xacro:unless>
       <parent link="${link_prefix}rocker_L_link"/>
       <child link="${link_prefix}wheel_FL_link"/>
@@ -160,5 +202,10 @@
     </joint>
     <joint name="${joint_prefix}wheel_RL_joint" type="continuous">
-      <origin xyz="0.15256 -0.08214 -0.08802" rpy="0 0 0"/>
+      <xacro:if value="${mecanum_wheels}">
+        <origin xyz="0.15256 -0.00884 -0.08802" rpy="0 0 0"/>
+      </xacro:if>
+      <xacro:unless value="${mecanum_wheels}">
+        <origin xyz="0.15256 -0.08214 -0.08802" rpy="0 0 0"/>
+      </xacro:unless>
       <parent link="${link_prefix}rocker_L_link"/>
       <child link="${link_prefix}wheel_RL_link"/>
@@ -168,5 +215,10 @@
     </joint>
     <joint name="${joint_prefix}wheel_FR_joint" type="continuous">
-      <origin xyz="0.15256 -0.08214 -0.08802" rpy="0 0 0"/>
+      <xacro:if value="${mecanum_wheels}">
+        <origin xyz="0.15256 -0.00884 -0.08802" rpy="0 0 0"/>
+      </xacro:if>
+      <xacro:unless value="${mecanum_wheels}">
+        <origin xyz="0.15256 -0.08214 -0.08802" rpy="0 0 0"/>
+      </xacro:unless>
       <parent link="${link_prefix}rocker_R_link"/>
       <child link="${link_prefix}wheel_FR_link"/>
@@ -176,5 +228,10 @@
     </joint>
     <joint name="${joint_prefix}wheel_RR_joint" type="continuous">
-      <origin xyz="-0.15256 -0.08214 -0.08802" rpy="0 0 0"/>
+      <xacro:if value="${mecanum_wheels}">
+        <origin xyz="-0.15256 -0.00884 -0.08802" rpy="0 0 0"/>
+      </xacro:if>
+      <xacro:unless value="${mecanum_wheels}">
+        <origin xyz="-0.15256 -0.08214 -0.08802" rpy="0 0 0"/>
+      </xacro:unless>
       <parent link="${link_prefix}rocker_R_link"/>
       <child link="${link_prefix}wheel_RR_link"/>
